Commit message: bolide model visualized correctly on rviz

File: voiture.xacro (robot description, xacro)
@@ -44,5 +44,5 @@
     <origin xyz="0.127 0 -0.02" rpy="0 0 0" />
     <geometry>
-      <mesh filename="package://course_ros2/urdf/meshes/ChevroletCamaroLight.stl" scale="0.000990 0.0009375 0.0009375"/>
+      <mesh filename="/urdf/meshes/ChevroletCamaroLight.stl" scale="0.000990 0.0009375 0.0009375"/>
     </geometry>
   </xacro:macro>
@@ -50,5 +50,5 @@
     <origin xyz="0 0 0" rpy="0 0 0" />
     <geometry>
-      <mesh filename="package://course_ros2/urdf/meshes/left_wheel.stl" />
+      <mesh filename="/urdf/meshes/left_wheel.stl" />
     </geometry>
   </xacro:macro>
@@ -56,5 +56,5 @@
     <origin xyz="0 0 0" rpy="0 0 0" />
     <geometry>
-      <mesh filename="package://course_ros2/urdf/meshes/right_wheel.stl" />
+      <mesh filename="/urdf/meshes/right_wheel.stl" />
     </geometry>
   </xacro:macro>
@@ -62,5 +62,5 @@
     <origin xyz="0 0 0" rpy="0 0 0" />
     <geometry>
-      <mesh filename="package://course_ros2/urdf/meshes/right_wheel.stl" />
+      <mesh filename="/urdf/meshes/right_wheel.stl" />
     </geometry>
   </xacro:macro>
@@ -68,5 +68,5 @@
     <origin xyz="0 0 0" rpy="0 0 0" />
     <geometry>
-      <mesh filename="package://course_ros2/urdf/meshes/right_wheel.stl" />
+      <mesh filename="/urdf/meshes/right_wheel.stl" />
     </geometry>
   </xacro:macro>
@@ -75,5 +75,5 @@
     <origin xyz="0 0 0" rpy="0 0 0" />
     <geometry>
-      <mesh filename="package://course_ros2/urdf/meshes/hinge.stl" />
+      <mesh filename="/urdf/meshes/hinge.stl" />
     </geometry>
   </xacro:macro>
@@ -81,5 +81,5 @@
     <origin xyz="0 0 0" rpy="0 0 0" />
     <geometry>
-      <mesh filename="package://course_ros2/urdf/meshes/hinge.stl" />
+      <mesh filename="/urdf/meshes/hinge.stl" />
     </geometry>
   </xacro:macro>
@@ -279,5 +279,5 @@
       <origin xyz="0 0 -0.011" rpy="0 0 0"/>
       <geometry>
-        <mesh filename="package://course_ros2/urdf/meshes/rplidar.stl"/>
+        <mesh filename="/urdf/meshes/rplidar.stl"/>
         <material name="grey" />
       </geometry>
